Commit message: (2020.06.20) (SOEM + Xenomai + Eigen + RBDL + Joint/Cartesian Control)

File: model/PONGBOT_ONE_LEG/urdf/PONGBOT_ONE_LEG.urdf (robot description, URDF)
Before this commit: robot PONGBOT_ONE_LEG, 5 links, 4 joints
Links:
- link BASE: mass 3.292 -> 3.6
- link CALF: mass 0.828 -> 0.35
- link HIP: mass 1.53 -> 2.35
- link THIGH: mass 3.306 -> 3.15
Joints:
- joint TIP_JOINT: axis 0.70711 0 0.70711 -> 0 0 0; type continuous -> fixed
